Commit message: hide isaac ros config

File: movensys_manipulator_description/urdf/movensys_manipulator.urdf (robot description, URDF)
Before this commit: robot manipulator, 14 links, 13 joints
Links:
- link Link0: geometry collision mesh filename=file:///home/admin/ws/install/movensys_manipulator_descript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; visual mesh filename=file:///home/admin/ws/install/movensys_manipulator_descript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
- link Link1: geometry collision mesh filename=file:///home/admin/ws/install/movensys_manipulator_descript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; visual mesh filename=file:///home/admin/ws/install/movensys_manipulator_descript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
- link Link2: geometry collision mesh filename=file:///home/admin/ws/install/movensys_manipulator_descript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; visual mesh filename=file:///home/admin/ws/install/movensys_manipulator_descript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
- link Link3: geometry collision mesh filename=file:///home/admin/ws/install/movensys_manipulator_descript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; visual mesh filename=file:///home/admin/ws/install/movensys_manipulator_descript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
- link Link4: geometry collision mesh filename=file:///home/admin/ws/install/movensys_manipulator_descript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; visual mesh filename=file:///home/admin/ws/install/movensys_manipulator_descript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
- link Link5: geometry collision mesh filename=file:///home/admin/ws/install/movensys_manipulator_descript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; visual mesh filename=file:///home/admin/ws/install/movensys_manipulator_descript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
- link Link6: geometry collision mesh filename=file:///home/admin/ws/install/movensys_manipulator_descript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; visual mesh filename=file:///home/admin/ws/install/movensys_manipulator_descript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
- link bracket: geometry collision mesh filename=file:///home/admin/ws/install/movensys_manipulator_descript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 scale=0.001 0.001 0.001; visual mesh filename=file:///home/admin/ws/install/movensys_manipulator_descript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 scale=0.001 0.001 0.001
- link gripper: geometry collision mesh filename=file:///home/admin/ws/install/movensys_manipulator_descript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 scale=0.001 0.001 0.001; visual mesh filename=file:///home/admin/ws/install/movensys_manipulator_descript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 scale=0.001 0.001 0.001
- link stand: geometry collision mesh filename=file:///home/admin/ws/install/movensys_manipulator_descript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 scale=0.001 0.001 0.001; visual mesh filename=file:///home/admin/ws/install/movensys_manipulator_descript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 scale=0.001 0.001 0.001
- link table: geometry collision mesh filename=file:///home/admin/ws/install/movensys_manipulator_descript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 scale=0.001 0.001 0.001; visual mesh filename=file:///home/admin/ws/install/movensys_manipulator_descript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 scale=0.001 0.001 0.001
Joints:
- joint joint1: limit lower=-3.14 upper=3.14 effort=50 velocity=3.0 -> lower=-3.14 upper=3.14 effort=50 velocity=1.0
- joint joint2: limit lower=-2.0 upper=2.0 effort=50 velocity=3.0 -> lower=-2.0 upper=2.0 effort=50 velocity=1.0
- joint joint3: limit lower=-0.2 upper=2.55 effort=50 velocity=3.0 -> lower=-0.2 upper=2.55 effort=50 velocity=1.0
- joint joint4: limit lower=-3.14 upper=3.14 effort=50 velocity=3.0 -> lower=-3.14 upper=3.14 effort=50 velocity=1.0
- joint joint5: limit lower=-2.5 upper=0.1 effort=50 velocity=3.0 -> lower=-2.5 upper=0.1 effort=50 velocity=1.0
- joint joint6: limit lower=-3.14 upper=3.14 effort=50 velocity=3.0 -> lower=-3.14 upper=3.14 effort=50 velocity=1.0
- joint picker_1_joint: limit lower=0.0 upper=0.045 effort=50 velocity=3.0 -> lower=0.0 upper=0.045 effort=50 velocity=1.0
- joint picker_2_joint: limit lower=0.0 upper=0.045 effort=50 velocity=3.0 -> lower=0.0 upper=0.045 effort=50 velocity=1.0

File: movensys_manipulator_description/urdf/movensys_manipulator.xacro (robot description, xacro)
@@ -2,5 +2,5 @@
 <robot name="manipulator" xmlns:xacro="http://www.ros.org/wiki/xacro">
     <xacro:include filename="$(find movensys_manipulator_description)/urdf/cr3a.xacro"/>
-    <xacro:cr3a prefix="" joint_vel="3.0" joint_effort="50"/>
+    <xacro:cr3a prefix="" joint_vel="1.0" joint_effort="50"/>
     <link name="world_manipulator"/>
     <joint name="world_manipulator_to_table" type="fixed">

Commit message: erase u stand

File: movensys_manipulator_description/urdf/movensys_manipulator.urdf (robot description, URDF)
Before this commit: robot manipulator, 14 links, 13 joints
Links:
- removed link stand
Joints:
- removed joint table_joint
- joint stand_joint: origin xyz=-0.03 0.275 0.265 rpy=0 0 0 -> xyz=-0.03 0.275 0.05 rpy=0 0 0; parent stand -> table

File: movensys_manipulator_description/urdf/movensys_manipulator.xacro (robot description, xacro)
@@ -32,35 +32,7 @@
         </collision>
     </link>
-    <joint name="table_joint" type="fixed">
-        <origin xyz="0 0 0" rpy="0 0 0"/>
+    <joint name="stand_joint" type="fixed">
+        <origin xyz="-0.03 0.275 0.05" rpy="0 0 0"/>
         <parent link="table"/>
-        <child link="stand"/>
-    </joint>
-    <link name="stand">
-        <inertial>
-        <origin xyz="0 0 0" rpy="0 0 0" />
-            <mass value="0.653" />
-            <inertia ixx="0.00075137" ixy="-3.0366E-08" ixz="1.2825E-06"
-                    iyy="0.00080094" iyz="2.5423E-09" izz="0.0010902" />
-        </inertial>
-        <visual>
-            <origin xyz="-0.23 -0.1 -1.285" rpy="0 0 0" />
-            <geometry>
-                <mesh filename="file://$(find movensys_manipulator_description)/urdf/assets/stand.STL" scale="0.001 0.001 0.001"/>
-            </geometry>
-            <material name="">
-                <color rgba="1 1 1 1" />
-            </material>
-        </visual>
-        <collision>
-            <origin xyz="-0.23 -0.1 -1.285" rpy="0 0 0" />
-            <geometry>
-                <mesh filename="file://$(find movensys_manipulator_description)/urdf/assets/stand.STL" scale="0.001 0.001 0.001"/>
-            </geometry>
-        </collision>
-    </link>
-    <joint name="stand_joint" type="fixed">
-        <origin xyz="-0.03 0.275 0.265" rpy="0 0 0"/>
-        <parent link="stand"/>
         <child link="Link0"/>
     </joint>
