Commit message: repair urdf

File: movensys_manipulator_description/urdf/cr3a.xacro (robot description, xacro)
@@ -28,5 +28,9 @@
       <axis xyz="0 0 1" />
       <limit lower="-3.14" upper="3.14" effort="${joint_effort}" velocity="${joint_vel}" />
-    </joint>
+      <dynamics damping="10.0" friction="1.0"/>
+    </joint>
+    <gazebo reference="${prefix}joint1">
+      <implicitSpringDamper>true</implicitSpringDamper>
+    </gazebo>
     <link name="${prefix}Link1">
       <inertial>
@@ -56,5 +60,9 @@
       <axis xyz="0 0 1" />
       <limit lower="-2.0" upper="2.0" effort="${joint_effort}" velocity="${joint_vel}" />
-    </joint>
+      <dynamics damping="15.0" friction="1.0"/>
+    </joint>
+    <gazebo reference="${prefix}joint2">
+      <implicitSpringDamper>true</implicitSpringDamper>
+    </gazebo>
     <link name="${prefix}Link2">
       <inertial>
@@ -84,5 +92,9 @@
       <axis xyz="0 0 1" />
       <limit lower="-0.2" upper="2.55" effort="${joint_effort}" velocity="${joint_vel}" />
-    </joint>
+      <dynamics damping="15.0" friction="1.0"/>
+    </joint>
+    <gazebo reference="${prefix}joint3">
+      <implicitSpringDamper>true</implicitSpringDamper>
+    </gazebo>
     <link name="${prefix}Link3">
       <inertial>
@@ -112,5 +124,9 @@
       <axis xyz="0 0 1" />
       <limit lower="-3.14" upper="3.14" effort="${joint_effort}" velocity="${joint_vel}" />
-    </joint>
+      <dynamics damping="10.0" friction="1.0"/>
+    </joint>
+    <gazebo reference="${prefix}joint4">
+      <implicitSpringDamper>true</implicitSpringDamper>
+    </gazebo>
     <link name="${prefix}Link4">
       <inertial>
@@ -140,5 +156,9 @@
       <axis xyz="0 0 1" />
       <limit lower="-2.5" upper="0.1" effort="${joint_effort}" velocity="${joint_vel}" />
-    </joint>
+      <dynamics damping="10.0" friction="1.0"/>
+    </joint>
+    <gazebo reference="${prefix}joint5">
+      <implicitSpringDamper>true</implicitSpringDamper>
+    </gazebo>
     <link name="${prefix}Link5">
       <inertial>
@@ -168,5 +188,9 @@
       <axis xyz="0 0 1" />
       <limit lower="-3.14" upper="3.14" effort="${joint_effort}" velocity="${joint_vel}" />
-    </joint>
+      <dynamics damping="5.0" friction="0.5"/>
+    </joint>
+    <gazebo reference="${prefix}joint6">
+      <implicitSpringDamper>true</implicitSpringDamper>
+    </gazebo>
     <link name="${prefix}Link6">
       <inertial>
@@ -247,5 +271,9 @@
       <axis xyz="-1 0 0"/>
       <limit effort="${joint_effort}" lower="0.0" upper="0.045" velocity="${joint_vel}" />
-    </joint>
+      <dynamics damping="5.0" friction="0.5"/>
+    </joint>
+    <gazebo reference="${prefix}picker_1_joint">
+      <implicitSpringDamper>true</implicitSpringDamper>
+    </gazebo>
     <link name="${prefix}picker_1">
       <inertial>
@@ -275,5 +303,9 @@
       <axis xyz="1 0 0" />
       <limit effort="${joint_effort}" lower="0.0" upper="0.045" velocity="${joint_vel}" />
-    </joint>
+      <dynamics damping="5.0" friction="0.5"/>
+    </joint>
+    <gazebo reference="${prefix}picker_2_joint">
+      <implicitSpringDamper>true</implicitSpringDamper>
+    </gazebo>
     <link name="${prefix}picker_2">
       <inertial>

File: movensys_manipulator_description/urdf/movensys_manipulator.urdf (robot description, URDF)
Before this commit: robot manipulator, 14 links, 13 joints
Joints:
- joint joint1: limit lower=-3.14 upper=3.14 effort=50 velocity=1.0 -> lower=-3.14 upper=3.14 effort=1000 velocity=1.0
- joint joint2: limit lower=-2.0 upper=2.0 effort=50 velocity=1.0 -> lower=-2.0 upper=2.0 effort=1000 velocity=1.0
- joint joint3: limit lower=-0.2 upper=2.55 effort=50 velocity=1.0 -> lower=-0.2 upper=2.55 effort=1000 velocity=1.0
- joint joint4: limit lower=-3.14 upper=3.14 effort=50 velocity=1.0 -> lower=-3.14 upper=3.14 effort=1000 velocity=1.0
- joint joint5: limit lower=-2.5 upper=0.1 effort=50 velocity=1.0 -> lower=-2.5 upper=0.1 effort=1000 velocity=1.0
- joint joint6: limit lower=-3.14 upper=3.14 effort=50 velocity=1.0 -> lower=-3.14 upper=3.14 effort=1000 velocity=1.0
- joint picker_1_joint: limit lower=0.0 upper=0.045 effort=50 velocity=1.0 -> lower=0.0 upper=0.045 effort=1000 velocity=1.0
- joint picker_2_joint: limit lower=0.0 upper=0.045 effort=50 velocity=1.0 -> lower=0.0 upper=0.045 effort=1000 velocity=1.0

Commit message: repair urdf

File: movensys_manipulator_description/urdf/cr3a.xacro (robot description, xacro)
@@ -214,33 +214,7 @@
       </collision>
     </link>
-    <joint name="${prefix}bracket_joint" type="fixed">
-      <origin xyz="0 0 0" rpy="0 0 0" />
+    <joint name="${prefix}gripper_joint" type="fixed">
+      <origin xyz="0 0 0" rpy="1.57 0 0" />
       <parent link="${prefix}Link6" />
-      <child link="${prefix}bracket" />
-    </joint>
-    <link name="${prefix}bracket">
-      <inertial>
-        <origin xyz="0.0585 0.037 0" rpy="0 0 3.14" />
-        <mass value="0.001" />
-        <inertia ixx="8.29484481057063E-05" ixy="-1.45209400395148E-09" ixz="-1.72340872805449E-11"
-                 iyy="8.35928339777967E-05" iyz="-1.33911019721127E-07" izz="0.000131911087085913" />
-      </inertial>
-      <visual>
-        <origin xyz="0.0585 0.037 0" rpy="0 0 3.14" />
-        <geometry>
-          <mesh filename="file://$(find movensys_manipulator_description)/urdf/assets/bracket.STL" scale="0.001 0.001 0.001"/>
-        </geometry>
-        <material name=""><color rgba="0 0 0 1" /></material>
-      </visual>
-      <collision>
-        <origin xyz="0.0585 0.037 0" rpy="0 0 3.14" />
-        <geometry>
-          <mesh filename="file://$(find movensys_manipulator_description)/urdf/assets/bracket.STL" scale="0.001 0.001 0.001"/>
-        </geometry>
-      </collision>
-    </link>
-    <joint name="${prefix}gripper_joint" type="fixed">
-      <origin xyz="0 0.003 0.003" rpy="1.57 0 0" />
-      <parent link="${prefix}bracket" />
       <child link="${prefix}gripper" />
     </joint>
@@ -253,5 +227,5 @@
       </inertial>
       <visual>
-        <origin xyz="-0.052 0.005 -0.09" rpy="0 0 0" />
+        <origin xyz="-0.052 0.0 -0.09" rpy="0 0 0" />
         <geometry>
           <mesh filename="file://$(find movensys_manipulator_description)/urdf/assets/gripper.STL" scale="0.001 0.001 0.001"/>
@@ -259,5 +233,5 @@
       </visual>
       <collision>
-        <origin xyz="-0.052 0.005 -0.09" rpy="0 0 0" />
+        <origin xyz="-0.052 0.0 -0.09" rpy="0 0 0" />
         <geometry>
           <mesh filename="file://$(find movensys_manipulator_description)/urdf/assets/gripper.STL" scale="0.001 0.001 0.001"/>

Commit message: rotate the robot

File: movensys_manipulator_description/urdf/cr3a.xacro (robot description, xacro)
@@ -27,5 +27,5 @@
       <child link="${prefix}Link1" />
       <axis xyz="0 0 1" />
-      <limit lower="-3.14" upper="3.14" effort="${joint_effort}" velocity="${joint_vel}" />
+      <limit lower="-1.57" upper="4.71239" effort="${joint_effort}" velocity="${joint_vel}" />
       <dynamics damping="10.0" friction="1.0"/>
     </joint>
@@ -59,5 +59,5 @@
       <child link="${prefix}Link2" />
       <axis xyz="0 0 1" />
-      <limit lower="-2.0" upper="2.0" effort="${joint_effort}" velocity="${joint_vel}" />
+      <limit lower="-1.57" upper="1.57" effort="${joint_effort}" velocity="${joint_vel}" />
       <dynamics damping="15.0" friction="1.0"/>
     </joint>
@@ -155,5 +155,5 @@
       <child link="${prefix}Link5" />
       <axis xyz="0 0 1" />
-      <limit lower="-2.5" upper="0.1" effort="${joint_effort}" velocity="${joint_vel}" />
+      <limit lower="-3.14" upper="0.1" effort="${joint_effort}" velocity="${joint_vel}" />
       <dynamics damping="10.0" friction="1.0"/>
     </joint>

File: movensys_manipulator_description/urdf/movensys_manipulator.xacro (robot description, xacro)
@@ -33,7 +33,51 @@
     </link>
     <joint name="stand_joint" type="fixed">
-        <origin xyz="-0.03 0.275 0.05" rpy="0 0 0"/>
+        <origin xyz="-0.03 0.275 0.05" rpy="0 0 -1.57"/>
         <parent link="table"/>
         <child link="Link0"/>
     </joint>
+    <link name="jetson_thor">
+        <visual>
+            <origin xyz="0 0 0" rpy="0 0 0"/>
+            <geometry>
+                <box size="0.2 0.2 0.07"/>
+            </geometry>
+            <material name="">
+                <color rgba="0.8 0.8 0.8 1"/>
+            </material>
+        </visual>
+        <collision>
+            <origin xyz="0 0 0" rpy="0 0 0"/>
+            <geometry>
+                <box size="0.2 0.2 0.07"/>
+            </geometry>
+        </collision>
+    </link>
+    <joint name="table_to_jetson_thor" type="fixed">
+        <parent link="table"/>
+        <child link="jetson_thor"/>
+        <origin xyz="0.36 0.18 0.07" rpy="0 0 0"/>
+    </joint>
+    <link name="power_supply">
+        <visual>
+            <origin xyz="0 0 0" rpy="0 0 0"/>
+            <geometry>
+                <box size="0.25 0.125 0.04"/>
+            </geometry>
+            <material name="">
+                <color rgba="0.8 0.8 0.8 1"/>
+            </material>
+        </visual>
+        <collision>
+            <origin xyz="0 0 0" rpy="0 0 0"/>
+            <geometry>
+                <box size="0.25 0.125  0.04"/>
+            </geometry>
+        </collision>
+    </link>
+    <joint name="table_to_power_supply" type="fixed">
+        <parent link="table"/>
+        <child link="power_supply"/>
+        <origin xyz="-0.3 0.2 0.065" rpy="0 0 1.57"/>
+    </joint>
 </robot>
