Commit message: add robot model selection in description

File: movensys_manipulator_description/urdf/dobot_cr3a/control.xacro (robot description, xacro)
@@ -65,5 +65,5 @@
 			<robot_param>robot_description</robot_param>
 			<robot_param_node>robot_state_publisher</robot_param_node>
-			<parameters>$(find movensys_manipulator_description)/urdf/control.yaml</parameters>
+			<parameters>$(find movensys_manipulator_description)/urdf/dobot_cr3a/control.yaml</parameters>
 		</plugin>
 	</gazebo>

File: movensys_manipulator_description/urdf/dobot_cr3a/dobot_cr3a.xacro (robot description, xacro)
@@ -1,6 +1,6 @@
 <?xml version="1.0"?>
 <robot xmlns:xacro="http://www.ros.org/wiki/xacro">
-  <xacro:macro name="cr3a" params="prefix joint_vel joint_effort">
-    <link name="${prefix}Link0">
+  <xacro:macro name="dobot_cr3a" params="joint_vel joint_effort">
+    <link name="Link0">
       <inertial>
         <origin xyz="-0.0027213 3.915E-07 0.022038" rpy="0 0 0" />
@@ -11,5 +11,5 @@
         <origin xyz="0 0 0" rpy="0 0 -1.57" />
         <geometry>
-          <mesh filename="file://$(find movensys_manipulator_description)/urdf/assets/Link0.STL" />
+          <mesh filename="file://$(find movensys_manipulator_description)/urdf/dobot_cr3a/assets/Link0.STL" />
         </geometry>
         <material name=""><color rgba="1 1 1 1" /></material>
@@ -18,20 +18,20 @@
         <origin xyz="0 0 0" rpy="0 0 -1.57" />
         <geometry>
-          <mesh filename="file://$(find movensys_manipulator_description)/urdf/assets/Link0.STL" />
-        </geometry>
-      </collision>
-    </link>
-    <joint name="${prefix}joint1" type="revolute">
+          <mesh filename="file://$(find movensys_manipulator_description)/urdf/dobot_cr3a/assets/Link0.STL" />
+        </geometry>
+      </collision>
+    </link>
+    <joint name="joint1" type="revolute">
       <origin xyz="0 0 0.1283" rpy="0 0 0" />
-      <parent link="${prefix}Link0" />
-      <child link="${prefix}Link1" />
+      <parent link="Link0" />
+      <child link="Link1" />
       <axis xyz="0 0 1" />
       <limit lower="-1.57" upper="4.71239" effort="${joint_effort}" velocity="${joint_vel}" />
       <dynamics damping="10.0" friction="1.0"/>
     </joint>
-    <gazebo reference="${prefix}joint1">
-      <implicitSpringDamper>true</implicitSpringDamper>
-    </gazebo>
-    <link name="${prefix}Link1">
+    <gazebo reference="joint1">
+      <implicitSpringDamper>true</implicitSpringDamper>
+    </gazebo>
+    <link name="Link1">
       <inertial>
         <origin xyz="-3.68657602416735E-05 -0.00394516685385322 0.00364037839421286" rpy="0 0 0" />
@@ -43,27 +43,27 @@
         <origin xyz="0 0 0" rpy="0 0 0" />
         <geometry>
-          <mesh filename="file://$(find movensys_manipulator_description)/urdf/assets/Link1.STL" />
-        </geometry>
-        <material name=""><color rgba="1 1 1 1" /></material>
-      </visual>
-      <collision>
-        <origin xyz="0 0 0" rpy="0 0 0" />
-        <geometry>
-          <mesh filename="file://$(find movensys_manipulator_description)/urdf/assets/Link1.STL" />
-        </geometry>
-      </collision>
-    </link>
-    <joint name="${prefix}joint2" type="revolute">
+          <mesh filename="file://$(find movensys_manipulator_description)/urdf/dobot_cr3a/assets/Link1.STL" />
+        </geometry>
+        <material name=""><color rgba="1 1 1 1" /></material>
+      </visual>
+      <collision>
+        <origin xyz="0 0 0" rpy="0 0 0" />
+        <geometry>
+          <mesh filename="file://$(find movensys_manipulator_description)/urdf/dobot_cr3a/assets/Link1.STL" />
+        </geometry>
+      </collision>
+    </link>
+    <joint name="joint2" type="revolute">
       <origin xyz="0 0 0" rpy="1.5708 1.5708 0" />
-      <parent link="${prefix}Link1" />
-      <child link="${prefix}Link2" />
+      <parent link="Link1" />
+      <child link="Link2" />
       <axis xyz="0 0 1" />
       <limit lower="-1.57" upper="1.57" effort="${joint_effort}" velocity="${joint_vel}" />
       <dynamics damping="15.0" friction="1.0"/>
     </joint>
-    <gazebo reference="${prefix}joint2">
-      <implicitSpringDamper>true</implicitSpringDamper>
-    </gazebo>
-    <link name="${prefix}Link2">
+    <gazebo reference="joint2">
+      <implicitSpringDamper>true</implicitSpringDamper>
+    </gazebo>
+    <link name="Link2">
       <inertial>
         <origin xyz="-0.129235280055448 1.440541622715E-05 0.133173619961293" rpy="0 0 0" />
@@ -75,27 +75,27 @@
         <origin xyz="0 0 0" rpy="0 0 0" />
         <geometry>
-          <mesh filename="file://$(find movensys_manipulator_description)/urdf/assets/Link2.STL" />
-        </geometry>
-        <material name=""><color rgba="1 1 1 1" /></material>
-      </visual>
-      <collision>
-        <origin xyz="0 0 0" rpy="0 0 0" />
-        <geometry>
-          <mesh filename="file://$(find movensys_manipulator_description)/urdf/assets/Link2.STL" />
-        </geometry>
-      </collision>
-    </link>
-    <joint name="${prefix}joint3" type="revolute">
+          <mesh filename="file://$(find movensys_manipulator_description)/urdf/dobot_cr3a/assets/Link2.STL" />
+        </geometry>
+        <material name=""><color rgba="1 1 1 1" /></material>
+      </visual>
+      <collision>
+        <origin xyz="0 0 0" rpy="0 0 0" />
+        <geometry>
+          <mesh filename="file://$(find movensys_manipulator_description)/urdf/dobot_cr3a/assets/Link2.STL" />
+        </geometry>
+      </collision>
+    </link>
+    <joint name="joint3" type="revolute">
       <origin xyz="-0.274 0 0" rpy="0 0 0" />
-      <parent link="${prefix}Link2" />
-      <child link="${prefix}Link3" />
+      <parent link="Link2" />
+      <child link="Link3" />
       <axis xyz="0 0 1" />
       <limit lower="-0.2" upper="2.55" effort="${joint_effort}" velocity="${joint_vel}" />
       <dynamics damping="15.0" friction="1.0"/>
     </joint>
-    <gazebo reference="${prefix}joint3">
-      <implicitSpringDamper>true</implicitSpringDamper>
-    </gazebo>
-    <link name="${prefix}Link3">
+    <gazebo reference="joint3">
+      <implicitSpringDamper>true</implicitSpringDamper>
+    </gazebo>
+    <link name="Link3">
       <inertial>
         <origin xyz="-0.119822632176479 8.63344146663093E-08 0.0099876637825216" rpy="0 0 0" />
@@ -107,27 +107,27 @@
         <origin xyz="0 0 0" rpy="0 0 0" />
         <geometry>
-          <mesh filename="file://$(find movensys_manipulator_description)/urdf/assets/Link3.STL" />
-        </geometry>
-        <material name=""><color rgba="1 1 1 1" /></material>
-      </visual>
-      <collision>
-        <origin xyz="0 0 0" rpy="0 0 0" />
-        <geometry>
-          <mesh filename="file://$(find movensys_manipulator_description)/urdf/assets/Link3.STL" />
-        </geometry>
-      </collision>
-    </link>
-    <joint name="${prefix}joint4" type="revolute">
+          <mesh filename="file://$(find movensys_manipulator_description)/urdf/dobot_cr3a/assets/Link3.STL" />
+        </geometry>
+        <material name=""><color rgba="1 1 1 1" /></material>
+      </visual>
+      <collision>
+        <origin xyz="0 0 0" rpy="0 0 0" />
+        <geometry>
+          <mesh filename="file://$(find movensys_manipulator_description)/urdf/dobot_cr3a/assets/Link3.STL" />
+        </geometry>
+      </collision>
+    </link>
+    <joint name="joint4" type="revolute">
       <origin xyz="-0.23 0 0.1283" rpy="0 0 -1.5708" />
-      <parent link="${prefix}Link3" />
-      <child link="${prefix}Link4" />
+      <parent link="Link3" />
+      <child link="Link4" />
       <axis xyz="0 0 1" />
       <limit lower="-3.14" upper="3.14" effort="${joint_effort}" velocity="${joint_vel}" />
       <dynamics damping="10.0" friction="1.0"/>
     </joint>
-    <gazebo reference="${prefix}joint4">
-      <implicitSpringDamper>true</implicitSpringDamper>
-    </gazebo>
-    <link name="${prefix}Link4">
+    <gazebo reference="joint4">
+      <implicitSpringDamper>true</implicitSpringDamper>
+    </gazebo>
+    <link name="Link4">
       <inertial>
         <origin xyz="1.74679534498573E-07 0.0034522361215461 -0.0028730999658578" rpy="0 0 0" />
@@ -139,27 +139,27 @@
         <origin xyz="0 0 0" rpy="0 0 0" />
         <geometry>
-          <mesh filename="file://$(find movensys_manipulator_description)/urdf/assets/Link4.STL" />
-        </geometry>
-        <material name=""><color rgba="1 1 1 1" /></material>
-      </visual>
-      <collision>
-        <origin xyz="0 0 0" rpy="0 0 0" />
-        <geometry>
-          <mesh filename="file://$(find movensys_manipulator_description)/urdf/assets/Link4.STL" />
-        </geometry>
-      </collision>
-    </link>
-    <joint name="${prefix}joint5" type="revolute">
+          <mesh filename="file://$(find movensys_manipulator_description)/urdf/dobot_cr3a/assets/Link4.STL" />
+        </geometry>
+        <material name=""><color rgba="1 1 1 1" /></material>
+      </visual>
+      <collision>
+        <origin xyz="0 0 0" rpy="0 0 0" />
+        <geometry>
+          <mesh filename="file://$(find movensys_manipulator_description)/urdf/dobot_cr3a/assets/Link4.STL" />
+        </geometry>
+      </collision>
+    </link>
+    <joint name="joint5" type="revolute">
       <origin xyz="0 -0.116 0" rpy="1.5708 0 0" />
-      <parent link="${prefix}Link4" />
-      <child link="${prefix}Link5" />
+      <parent link="Link4" />
+      <child link="Link5" />
       <axis xyz="0 0 1" />
       <limit lower="-3.14" upper="0.1" effort="${joint_effort}" velocity="${joint_vel}" />
       <dynamics damping="10.0" friction="1.0"/>
     </joint>
-    <gazebo reference="${prefix}joint5">
-      <implicitSpringDamper>true</implicitSpringDamper>
-    </gazebo>
-    <link name="${prefix}Link5">
+    <gazebo reference="joint5">
+      <implicitSpringDamper>true</implicitSpringDamper>
+    </gazebo>
+    <link name="Link5">
       <inertial>
         <origin xyz="-1.74603758796282E-07 -0.00333192403958193 -0.00286780844130663" rpy="0 0 0" />
@@ -171,27 +171,27 @@
         <origin xyz="0 0 0" rpy="0 0 0" />
         <geometry>
-          <mesh filename="file://$(find movensys_manipulator_description)/urdf/assets/Link5.STL" />
-        </geometry>
-        <material name=""><color rgba="1 1 1 1" /></material>
-      </visual>
-      <collision>
-        <origin xyz="0 0 0" rpy="0 0 0" />
-        <geometry>
-          <mesh filename="file://$(find movensys_manipulator_description)/urdf/assets/Link5.STL" />
-        </geometry>
-      </collision>
-    </link>
-    <joint name="${prefix}joint6" type="revolute">
+          <mesh filename="file://$(find movensys_manipulator_description)/urdf/dobot_cr3a/assets/Link5.STL" />
+        </geometry>
+        <material name=""><color rgba="1 1 1 1" /></material>
+      </visual>
+      <collision>
+        <origin xyz="0 0 0" rpy="0 0 0" />
+        <geometry>
+          <mesh filename="file://$(find movensys_manipulator_description)/urdf/dobot_cr3a/assets/Link5.STL" />
+        </geometry>
+      </collision>
+    </link>
+    <joint name="joint6" type="revolute">
       <origin xyz="0 0.105 0" rpy="-1.5708 0 0" />
-      <parent link="${prefix}Link5" />
-      <child link="${prefix}Link6" />
+      <parent link="Link5" />
+      <child link="Link6" />
       <axis xyz="0 0 1" />
       <limit lower="-3.14" upper="3.14" effort="${joint_effort}" velocity="${joint_vel}" />
       <dynamics damping="5.0" friction="0.5"/>
     </joint>
-    <gazebo reference="${prefix}joint6">
-      <implicitSpringDamper>true</implicitSpringDamper>
-    </gazebo>
-    <link name="${prefix}Link6">
+    <gazebo reference="joint6">
+      <implicitSpringDamper>true</implicitSpringDamper>
+    </gazebo>
+    <link name="Link6">
       <inertial>
         <origin xyz="-5.77233004964394E-07 0.000270130842674243 -0.0201386770129675" rpy="0 0 0" />
@@ -203,101 +203,12 @@
         <origin xyz="0 0 0" rpy="0 0 0" />
         <geometry>
-          <mesh filename="file://$(find movensys_manipulator_description)/urdf/assets/Link6.STL" />
-        </geometry>
-        <material name=""><color rgba="1 1 1 1" /></material>
-      </visual>
-      <collision>
-        <origin xyz="0 0 0" rpy="0 0 0" />
-        <geometry>
-          <mesh filename="file://$(find movensys_manipulator_description)/urdf/assets/Link6.STL" />
-        </geometry>
-      </collision>
-    </link>
-    <joint name="${prefix}gripper_joint" type="fixed">
-      <origin xyz="0 0 0" rpy="1.57 0 0" />
-      <parent link="${prefix}Link6" />
-      <child link="${prefix}gripper" />
-    </joint>
-    <link name="${prefix}gripper">
-      <inertial>
-        <origin xyz="0 0 0" rpy="0 0 0" />
-        <mass value="1.0" />
-        <inertia ixx="8.29484481057063E-05" ixy="-1.45209400395148E-09" ixz="-1.72340872805449E-11"
-                 iyy="8.35928339777967E-05" iyz="-1.33911019721127E-07" izz="0.000131911087085913" />
-      </inertial>
-      <visual>
-        <origin xyz="-0.052 0.0 -0.09" rpy="0 0 0" />
-        <geometry>
-          <mesh filename="file://$(find movensys_manipulator_description)/urdf/assets/gripper.STL" scale="0.001 0.001 0.001"/>
-        </geometry>
-      </visual>
-      <collision>
-        <origin xyz="-0.052 0.0 -0.09" rpy="0 0 0" />
-        <geometry>
-          <mesh filename="file://$(find movensys_manipulator_description)/urdf/assets/gripper.STL" scale="0.001 0.001 0.001"/>
-        </geometry>
-      </collision>
-    </link>
-    <joint name="${prefix}picker_1_joint" type="prismatic">
-      <origin xyz="0.05 0.175 0.004" rpy="0 0 0" />
-      <parent link="${prefix}gripper" />
-      <child link="${prefix}picker_1" />
-      <axis xyz="-1 0 0"/>
-      <limit effort="${joint_effort}" lower="0.0" upper="0.045" velocity="${joint_vel}" />
-      <dynamics damping="5.0" friction="0.5"/>
-    </joint>
-    <gazebo reference="${prefix}picker_1_joint">
-      <implicitSpringDamper>true</implicitSpringDamper>
-    </gazebo>
-    <link name="${prefix}picker_1">
-      <inertial>
-        <origin xyz="0 0 0" rpy="0 0 0" />
-        <mass value="0.1" />
-        <inertia ixx="8.29484481057063E-05" ixy="-1.45209400395148E-09" ixz="-1.72340872805449E-11"
-                 iyy="8.35928339777967E-05" iyz="-1.33911019721127E-07" izz="0.000131911087085913" />
-      </inertial>
-      <visual>
-        <origin xyz="0 0 0" rpy="0 0 0" />
-          <geometry>
-            <box size="0.005 0.04 0.02"></box>
-          </geometry>
-        <material name=""><color rgba="1 1 1 1" /></material>
-      </visual>
-      <collision>
-        <origin xyz="0 0 0" rpy="0 0 0" />
-          <geometry>
-            <box size="0.005 0.04 0.02"></box>
-          </geometry>
-      </collision>
-    </link>
-    <joint name="${prefix}picker_2_joint" type="prismatic">
-      <origin xyz="-0.05 0.175 0.004" rpy="0 0 0" />
-      <parent link="${prefix}gripper" />
-      <child link="${prefix}picker_2" />
-      <axis xyz="1 0 0" />
-      <limit effort="${joint_effort}" lower="0.0" upper="0.045" velocity="${joint_vel}" />
-      <dynamics damping="5.0" friction="0.5"/>
-    </joint>
-    <gazebo reference="${prefix}picker_2_joint">
-      <implicitSpringDamper>true</implicitSpringDamper>
-    </gazebo>
-    <link name="${prefix}picker_2">
-      <inertial>
-        <origin xyz="1 0 0" rpy="0 0 0" />
-        <mass value="0.1" />
-        <inertia ixx="8.29484481057063E-05" ixy="-1.45209400395148E-09" ixz="-1.72340872805449E-11"
-                 iyy="8.35928339777967E-05" iyz="-1.33911019721127E-07" izz="0.000131911087085913" />
-      </inertial>
-      <visual>
-        <origin xyz="0 0 0" rpy="0 0 0" />
-        <geometry>
-          <box size="0.005 0.04 0.02"></box>
-        </geometry>
-        <material name=""><color rgba="1 1 1 1" /></material>
-      </visual>
-      <collision>
-        <origin xyz="0 0 0" rpy="0 0 0" />
-        <geometry>
-          <box size="0.005 0.04 0.02"></box>
+          <mesh filename="file://$(find movensys_manipulator_description)/urdf/dobot_cr3a/assets/Link6.STL" />
+        </geometry>
+        <material name=""><color rgba="1 1 1 1" /></material>
+      </visual>
+      <collision>
+        <origin xyz="0 0 0" rpy="0 0 0" />
+        <geometry>
+          <mesh filename="file://$(find movensys_manipulator_description)/urdf/dobot_cr3a/assets/Link6.STL" />
         </geometry>
       </collision>

File: movensys_manipulator_description/urdf/dobot_cr3a/stage.xacro (robot description, xacro)
@@ -1,12 +1,5 @@
 <?xml version="1.0"?>
-<robot name="manipulator" xmlns:xacro="http://www.ros.org/wiki/xacro">
-    <xacro:include filename="$(find movensys_manipulator_description)/urdf/cr3a.xacro"/>
-    <xacro:cr3a prefix="" joint_vel="1.0" joint_effort="1000"/>
-    <link name="world_manipulator"/>
-    <joint name="world_manipulator_to_table" type="fixed">
-        <parent link="world_manipulator"/>
-        <child  link="table"/>
-        <origin xyz="0 0 0" rpy="0 0 0"/>
-    </joint>
+<robot xmlns:xacro="http://www.ros.org/wiki/xacro">
+  <xacro:macro name="stage">
     <link name="table">
         <inertial>
@@ -19,5 +12,5 @@
             <origin xyz="-0.5 -0.35 -1.285" rpy="0 0 0" />
             <geometry>
-                <mesh filename="file://$(find movensys_manipulator_description)/urdf/assets/table.STL" scale="0.001 0.001 0.001"/>
+                <mesh filename="file://$(find movensys_manipulator_description)/urdf/dobot_cr3a/assets/table.STL" scale="0.001 0.001 0.001"/>
             </geometry>
             <material name="">
@@ -28,13 +21,8 @@
             <origin xyz="-0.5 -0.35 -1.285" rpy="0 0 0" />
             <geometry>
-                <mesh filename="file://$(find movensys_manipulator_description)/urdf/assets/table.STL" scale="0.001 0.001 0.001"/>
+                <mesh filename="file://$(find movensys_manipulator_description)/urdf/dobot_cr3a/assets/table.STL" scale="0.001 0.001 0.001"/>
             </geometry>
         </collision>
     </link>
-    <joint name="stand_joint" type="fixed">
-        <origin xyz="-0.03 0.275 0.05" rpy="0 0 -1.57"/>
-        <parent link="table"/>
-        <child link="Link0"/>
-    </joint>
     <link name="jetson_thor">
         <visual>
@@ -81,3 +69,4 @@
         <origin xyz="-0.3 0.2 0.065" rpy="0 0 1.57"/>
     </joint>
+  </xacro:macro>
 </robot>
