Commit message: fix gazebo cr3a

File: movensys_manipulator_description/urdf/dobot_cr3a/movensys_manipulator.gazebo.xacro (robot description, xacro)
@@ -4,3 +4,8 @@
   <xacro:include filename="$(find movensys_manipulator_description)/urdf/dobot_cr3a/control.xacro"/>
   <xacro:include filename="$(find movensys_manipulator_description)/urdf/dobot_cr3a/transmission.xacro"/>
+  <link name="world"/>
+  <joint name="world_fixed" type="fixed">
+    <parent link="world"/>
+    <child link="world_manipulator"/>
+  </joint>
 </robot>
