Commit message: use local urdf

File: movensys_manipulator_description/urdf/dobot_cr3a/movensys_manipulator.urdf (robot description, URDF)
Before this commit: robot manipulator, 14 links, 13 joints
Links:
- link Link0: geometry collision mesh filename=file:///home/hehe-jazzy/workspaces/movensys_ws/install/move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; visual mesh filename=file:///home/hehe-jazzy/workspaces/movensys_ws/install/move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
- link Link1: geometry collision mesh filename=file:///home/hehe-jazzy/workspaces/movensys_ws/install/move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; visual mesh filename=file:///home/hehe-jazzy/workspaces/movensys_ws/install/move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
- link Link2: geometry collision mesh filename=file:///home/hehe-jazzy/workspaces/movensys_ws/install/move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; visual mesh filename=file:///home/hehe-jazzy/workspaces/movensys_ws/install/move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
- link Link3: geometry collision mesh filename=file:///home/hehe-jazzy/workspaces/movensys_ws/install/move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; visual mesh filename=file:///home/hehe-jazzy/workspaces/movensys_ws/install/move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
- link Link4: geometry collision mesh filename=file:///home/hehe-jazzy/workspaces/movensys_ws/install/move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; visual mesh filename=file:///home/hehe-jazzy/workspaces/movensys_ws/install/move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
- link Link5: geometry collision mesh filename=file:///home/hehe-jazzy/workspaces/movensys_ws/install/move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; visual mesh filename=file:///home/hehe-jazzy/workspaces/movensys_ws/install/move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
- link Link6: geometry collision mesh filename=file:///home/hehe-jazzy/workspaces/movensys_ws/install/move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; visual mesh filename=file:///home/hehe-jazzy/workspaces/movensys_ws/install/move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
- link bracket: geometry collision mesh filename=file:///home/hehe-jazzy/workspaces/movensys_ws/install/move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 scale=0.001 0.001 0.001; visual mesh filename=file:///home/hehe-jazzy/workspaces/movensys_ws/install/move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 scale=0.001 0.001 0.001
- link gripper: geometry collision mesh filename=file:///home/hehe-jazzy/workspaces/movensys_ws/install/move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 scale=0.001 0.001 0.001; visual mesh filename=file:///home/hehe-jazzy/workspaces/movensys_ws/install/move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 scale=0.001 0.001 0.001
- link table: geometry collision mesh filename=file:///home/hehe-jazzy/workspaces/movensys_ws/install/move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 scale=0.001 0.001 0.001; visual mesh filename=file:///home/hehe-jazzy/workspaces/movensys_ws/install/move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 scale=0.001 0.001 0.001
