Commit message: repair workdir

File: movensys_manipulator_description/urdf/dobot_cr3a/dobot_cr3a.xacro (robot description, xacro)
@@ -27,5 +27,5 @@
       <child link="Link1" />
       <axis xyz="0 0 1" />
-      <limit lower="-1.57" upper="4.71239" effort="${joint_effort}" velocity="${joint_vel}" />
+      <limit lower="-0.2" upper="6.0" effort="${joint_effort}" velocity="${joint_vel}" />
       <dynamics damping="10.0" friction="1.0"/>
     </joint>

Commit message: repair joint limit

File: movensys_manipulator_description/urdf/dobot_cr3a/dobot_cr3a.xacro (robot description, xacro)
@@ -123,5 +123,5 @@
       <child link="Link4" />
       <axis xyz="0 0 1" />
-      <limit lower="-3.14" upper="3.14" effort="${joint_effort}" velocity="${joint_vel}" />
+      <limit lower="-2.5" upper="2.5" effort="${joint_effort}" velocity="${joint_vel}" />
       <dynamics damping="10.0" friction="1.0"/>
     </joint>

File: movensys_manipulator_description/urdf/dobot_cr5a/dobot_cr5a.xacro (robot description, xacro)
@@ -196,5 +196,5 @@
       <child link="Link4" />
       <axis xyz="0 0 1" />
-      <limit lower="-3.14" upper="3.14" effort="${joint_effort}" velocity="${joint_vel}" />
+      <limit lower="-2.5" upper="2.5" effort="${joint_effort}" velocity="${joint_vel}" />
       <dynamics damping="10.0" friction="1.0"/>
     </joint>

Commit message: repair joint limit

File: movensys_manipulator_description/urdf/dobot_cr3a/dobot_cr3a.xacro (robot description, xacro)
@@ -27,5 +27,5 @@
       <child link="Link1" />
       <axis xyz="0 0 1" />
-      <limit lower="-0.2" upper="6.0" effort="${joint_effort}" velocity="${joint_vel}" />
+      <limit lower="-3.0" upper="3.0" effort="${joint_effort}" velocity="${joint_vel}" />
       <dynamics damping="10.0" friction="1.0"/>
     </joint>
@@ -91,5 +91,5 @@
       <child link="Link3" />
       <axis xyz="0 0 1" />
-      <limit lower="-0.2" upper="2.55" effort="${joint_effort}" velocity="${joint_vel}" />
+      <limit lower="-2.55" upper="0.2" effort="${joint_effort}" velocity="${joint_vel}" />
       <dynamics damping="15.0" friction="1.0"/>
     </joint>
@@ -155,5 +155,5 @@
       <child link="Link5" />
       <axis xyz="0 0 1" />
-      <limit lower="-3.14" upper="0.1" effort="${joint_effort}" velocity="${joint_vel}" />
+      <limit lower="-0.1" upper="3.0" effort="${joint_effort}" velocity="${joint_vel}" />
       <dynamics damping="10.0" friction="1.0"/>
     </joint>
@@ -187,5 +187,5 @@
       <child link="Link6" />
       <axis xyz="0 0 1" />
-      <limit lower="-3.14" upper="3.14" effort="${joint_effort}" velocity="${joint_vel}" />
+      <limit lower="-3.0" upper="3.0" effort="${joint_effort}" velocity="${joint_vel}" />
       <dynamics damping="5.0" friction="0.5"/>
     </joint>

File: movensys_manipulator_description/urdf/dobot_cr3a/stage.xacro (robot description, xacro)
@@ -47,26 +47,4 @@
         <origin xyz="0.36 0.18 0.07" rpy="0 0 0"/>
     </joint>
-    <link name="power_supply">
-        <visual>
-            <origin xyz="0 0 0" rpy="0 0 0"/>
-            <geometry>
-                <box size="0.25 0.125 0.04"/>
-            </geometry>
-            <material name="">
-                <color rgba="0.8 0.8 0.8 1"/>
-            </material>
-        </visual>
-        <collision>
-            <origin xyz="0 0 0" rpy="0 0 0"/>
-            <geometry>
-                <box size="0.25 0.125  0.04"/>
-            </geometry>
-        </collision>
-    </link>
-    <joint name="table_to_power_supply" type="fixed">
-        <parent link="table"/>
-        <child link="power_supply"/>
-        <origin xyz="-0.3 0.2 0.065" rpy="0 0 1.57"/>
-    </joint>
   </xacro:macro>
 </robot>

Commit message: safe joint coverage

File: movensys_manipulator_description/urdf/dobot_cr3a/dobot_cr3a.xacro (robot description, xacro)
@@ -59,5 +59,5 @@
       <child link="Link2" />
       <axis xyz="0 0 1" />
-      <limit lower="-1.57" upper="1.57" effort="${joint_effort}" velocity="${joint_vel}" />
+      <limit lower="-1.57" upper="1.1" effort="${joint_effort}" velocity="${joint_vel}" />
       <dynamics damping="15.0" friction="1.0"/>
     </joint>
