Commit message: fix cr5a urdf

File: movensys_manipulator_description/urdf/dobot_cr5a/movensys_manipulator.urdf (robot description, URDF)
Before this commit: robot manipulator, 9 links, 8 joints
Joints:
- joint robot_joint: origin xyz=-0.03 0.275 0.05 rpy=0 0 -1.57 -> xyz=0.25 0 0 rpy=0 0 1.57

File: movensys_manipulator_description/urdf/dobot_cr5a/movensys_manipulator.xacro (robot description, xacro)
@@ -11,5 +11,5 @@
     <xacro:stage />
     <joint name="robot_joint" type="fixed">
-        <origin xyz="0 0 0" rpy="0 0 0"/>
+        <origin xyz="0.25 0 0" rpy="0 0 1.57"/>
         <parent link="table"/>
         <child link="Link0"/>
