Commit message: add cr5a urdf

File: movensys_manipulator_description/urdf/dobot_cr5a/control.xacro (robot description, xacro)
@@ -30,34 +30,34 @@
 	    		<state_interface name="velocity"/>
 	    	</joint>
-		<joint name="joint3">
-	    		<command_interface name="position"/>
-	    		<state_interface name="position"/>
-	    		<state_interface name="velocity"/>
-	    	</joint>
-		<joint name="joint4">
-	    		<command_interface name="position"/>
-	    		<state_interface name="position"/>
-	    		<state_interface name="velocity"/>
-	    	</joint>
-		<joint name="joint5">
-	    		<command_interface name="position"/>
-	    		<state_interface name="position"/>
-	    		<state_interface name="velocity"/>
-	    	</joint>
-		<joint name="joint6">
-	    		<command_interface name="position"/>
-	    		<state_interface name="position"/>
-	    		<state_interface name="velocity"/>
-	    	</joint>
-		<joint name="picker_1_joint">
-	    		<command_interface name="position"/>
-	    		<state_interface name="position"/>
-	    		<state_interface name="velocity"/>
-	    	</joint>
-		<joint name="picker_2_joint">
-	    		<command_interface name="position"/>
-	    		<state_interface name="position"/>
-	    		<state_interface name="velocity"/>
-	    	</joint>
+			<joint name="joint3">
+					<command_interface name="position"/>
+					<state_interface name="position"/>
+					<state_interface name="velocity"/>
+				</joint>
+			<joint name="joint4">
+					<command_interface name="position"/>
+					<state_interface name="position"/>
+					<state_interface name="velocity"/>
+				</joint>
+			<joint name="joint5">
+					<command_interface name="position"/>
+					<state_interface name="position"/>
+					<state_interface name="velocity"/>
+				</joint>
+			<joint name="joint6">
+					<command_interface name="position"/>
+					<state_interface name="position"/>
+					<state_interface name="velocity"/>
+				</joint>
+			<joint name="picker_1_joint">
+					<command_interface name="position"/>
+					<state_interface name="position"/>
+					<state_interface name="velocity"/>
+				</joint>
+			<joint name="picker_2_joint">
+					<command_interface name="position"/>
+					<state_interface name="position"/>
+					<state_interface name="velocity"/>
+				</joint>
 	  	</ros2_control>
 	<gazebo>

File: movensys_manipulator_description/urdf/dobot_cr5a/movensys_manipulator.xacro (robot description, xacro)
@@ -11,5 +11,5 @@
     <xacro:stage />
     <joint name="robot_joint" type="fixed">
-        <origin xyz="-0.03 0.275 0.05" rpy="0 0 -1.57"/>
+        <origin xyz="0 0 0" rpy="0 0 0"/>
         <parent link="table"/>
         <child link="Link0"/>

File: movensys_manipulator_description/urdf/dobot_cr5a/stage.xacro (robot description, xacro)
@@ -10,7 +10,8 @@
         </inertial>
         <visual>
-            <origin xyz="-0.5 -0.35 -1.285" rpy="0 0 0" />
+            <origin xyz="0 0 0" rpy="0 0 0" />
             <geometry>
-                <box size="1.0 0.7 0.05"/>
+                <box size="1.0 0.7 0.01"/>
+            </geometry>
             <material name="">
                 <color rgba="1 1 1 1" />
@@ -18,5 +19,5 @@
         </visual>
         <collision>
-            <origin xyz="-0.5 -0.35 -1.285" rpy="0 0 0" />
+            <origin xyz="0 0 0" rpy="0 0 0" />
             <geometry>
                 <box size="1.0 0.7 0.05"/>

Commit message: delete picker

File: movensys_manipulator_description/urdf/dobot_cr5a/control.xacro (robot description, xacro)
@@ -50,14 +50,4 @@
 					<state_interface name="velocity"/>
 				</joint>
-			<joint name="picker_1_joint">
-					<command_interface name="position"/>
-					<state_interface name="position"/>
-					<state_interface name="velocity"/>
-				</joint>
-			<joint name="picker_2_joint">
-					<command_interface name="position"/>
-					<state_interface name="position"/>
-					<state_interface name="velocity"/>
-				</joint>
 	  	</ros2_control>
 	<gazebo>

File: movensys_manipulator_description/urdf/dobot_cr5a/movensys_manipulator.urdf (robot description, URDF)
Before this commit: robot manipulator, 9 links, 8 joints
Links:
- link Link0: geometry collision mesh filename=file:///home/admin/workspaces/movensys_ws/install/movensys_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; visual mesh filename=file:///home/admin/workspaces/movensys_ws/install/movensys_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
- link Link1: geometry collision mesh filename=file:///home/admin/workspaces/movensys_ws/install/movensys_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; visual mesh filename=file:///home/admin/workspaces/movensys_ws/install/movensys_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
- link Link2: geometry collision mesh filename=file:///home/admin/workspaces/movensys_ws/install/movensys_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; visual mesh filename=file:///home/admin/workspaces/movensys_ws/install/movensys_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
- link Link3: geometry collision mesh filename=file:///home/admin/workspaces/movensys_ws/install/movensys_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; visual mesh filename=file:///home/admin/workspaces/movensys_ws/install/movensys_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
- link Link4: geometry collision mesh filename=file:///home/admin/workspaces/movensys_ws/install/movensys_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; visual mesh filename=file:///home/admin/workspaces/movensys_ws/install/movensys_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
- link Link5: geometry collision mesh filename=file:///home/admin/workspaces/movensys_ws/install/movensys_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; visual mesh filename=file:///home/admin/workspaces/movensys_ws/install/movensys_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
- link Link6: geometry collision mesh filename=file:///home/admin/workspaces/movensys_ws/install/movensys_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; visual mesh filename=file:///home/admin/workspaces/movensys_ws/install/movensys_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
Joints:
- joint joint4: limit lower=-3.14 upper=3.14 effort=1000 velocity=3.0 -> lower=-2.5 upper=2.5 effort=1000 velocity=3.0

File: movensys_manipulator_description/urdf/dobot_cr5a/transmission.xacro (robot description, xacro)
@@ -61,23 +61,3 @@
     </actuator>
   </transmission>
-  <transmission name="picker_1_joint_transmission" type="SimpleTransmission">
-    <type>transmission_interface/SimpleTransmission</type>
-    <joint name="picker_1_joint">
-      <hardwareInterface>hardware_interface/PositionJointInterface</hardwareInterface>
-    </joint>
-    <actuator name="picker_1_joint_motor">
-      <hardwareInterface>hardware_interface/PositionJointInterface</hardwareInterface>
-      <mechanicalReduction>1</mechanicalReduction>
-    </actuator>
-  </transmission>
-  <transmission name="picker_2_joint_transmission" type="SimpleTransmission">
-    <type>transmission_interface/SimpleTransmission</type>
-    <joint name="picker_2_joint">
-      <hardwareInterface>hardware_interface/PositionJointInterface</hardwareInterface>
-    </joint>
-    <actuator name="picker_2_joint_motor">
-      <hardwareInterface>hardware_interface/PositionJointInterface</hardwareInterface>
-      <mechanicalReduction>1</mechanicalReduction>
-    </actuator>
-  </transmission>
 </robot>
